Commit message: Rebase from 'release/kinetic/uuv_gazebo_ros_plugins'

File: test/models/thrusters/model.xacro (robot description, xacro)
@@ -13,7 +13,15 @@
 -->
 <robot name="rexrov" xmlns:xacro="http://www.ros.org/wiki/xacro" >
-  <xacro:include filename="$(find uuv_descriptions)/models/common/urdf/common.urdf.xacro"/>
   <xacro:include filename="$(find uuv_gazebo_ros_plugins)/urdf/thruster_snippets.xacro"/>
-  <xacro:property name="prop_mesh_file" value="file://$(find uuv_descriptions)/models/rexrov/mesh/prop.dae"/>
+  <xacro:property name="prop_mesh_file" value="file://$(find uuv_descriptions)/mesh/prop.dae"/>
+  <xacro:macro name="box_inertial" params="x y z mass *origin">
+    <inertial>
+      <mass value="${mass}" />
+      <xacro:insert_block name="origin" />
+      <inertia ixx="${0.0833333 * mass * (y*y + z*z)}" ixy="0.0" ixz="0.0"
+             iyy="${0.0833333 * mass * (x*x + z*z)}" iyz="0.0"
+             izz="${0.0833333 * mass * (x*x + y*y)}" />
+    </inertial>
+  </xacro:macro>
   <link name="vehicle/base_link">
     <inertial>
